File: he_kbd/he_kbd.kicad_pcb (KiCad board)
At the start: 2 copper layers, 162.2 x 126.5 mm, 175 parts

Commit message: more pcb routing
Routing:
- net /hesig1: track 0.00 -> 64.3 mm, vias 0 -> 1
- net /hesig2: track 0.00 -> 42.9 mm, vias 0 -> 1
- net Net-(D11-DOUT): track 0.00 -> 24.8 mm
- net Net-(D2-DOUT): track 0.00 -> 22.7 mm
- net Net-(D7-DOUT): track 0.00 -> 19.6 mm, vias 0 -> 2
- net Net-(D8-DOUT): track 33.8 -> 29.0 mm
- net Net-(D13-DOUT): track 29.1 -> 27.3 mm, vias 2 -> 0
- net Net-(D1-DOUT): track 17.8 -> 19.6 mm, vias 2 -> 0
- net NEOPIXEL_POWER: track 841.9 -> 840.5 mm
- net Net-(D12-DOUT): track 27.3 -> 26.4 mm, vias 2 -> 0
- net Net-(D15-DOUT): vias 2 -> 0

Commit message: routing continued
Parts:
- moved R8 9.79 mm to (71.3, 75.7), turned to 0 degrees
- moved C24 6.23 mm to (31.3, 93.0)
- moved C28 6.20 mm to (90.5, 67.1), turned to 90 degrees
- moved C23 6.13 mm to (53.0, 93.1)
- moved C22 6.05 mm to (71.8, 88.6)
- moved C27 5.40 mm to (71.4, 69.5)
- moved AM1 1.67 mm to (78.3, 73.5)
Routing:
- net /hesig8: track 0.00 -> 87.4 mm, vias 0 -> 1
- net /hesig7: track 0.00 -> 84.1 mm, vias 0 -> 1
- net /hesig15: track 0.00 -> 80.9 mm, vias 0 -> 1
- net /hesig16: track 0.00 -> 77.0 mm, vias 0 -> 3
- net /hesig22: track 0.00 -> 66.7 mm, vias 0 -> 1
- net /hesig6: track 0.00 -> 64.3 mm, vias 0 -> 1
- net /hesig9: track 0.00 -> 61.6 mm, vias 0 -> 1
- net /hesig14: track 0.00 -> 60.3 mm, vias 0 -> 1
- net /hesig23: track 0.00 -> 58.9 mm, vias 0 -> 1
- net /hesig17: track 0.00 -> 58.7 mm, vias 0 -> 1
- net /hesig5: track 0.00 -> 43.1 mm, vias 0 -> 1
- net /hesig13: track 0.00 -> 42.7 mm, vias 0 -> 1
- net /hesig21: track 0.00 -> 42.5 mm, vias 0 -> 1
- net /hesig10: track 0.00 -> 40.7 mm, vias 0 -> 1
- net /hesig18: track 0.00 -> 39.2 mm, vias 0 -> 1
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
Commit message: mostly done routing ?!
Parts:
- C45: moved to F.Cu
- moved HE_37 81.7 mm to (72.3, 5.07), turned to 0 degrees
- moved HE_36 80.3 mm to (72.3, 0.44), turned to 0 degrees
- moved HE_40 78.7 mm to (72.3, 18.9), turned to 0 degrees
- moved C45 78.1 mm to (76.9, -0.70), turned to 0 degrees
- moved HE_39 76.3 mm to (72.3, 14.3), turned to 0 degrees
- moved HE_38 73.9 mm to (72.3, 9.69), turned to 0 degrees
- moved R9 6.56 mm to (97.0, 114.3), turned to -90 degrees
- moved C30 4.99 mm to (127.3, 71.5)
- moved C34 4.58 mm to (89.1, 48.0), turned to -90 degrees
- moved C32 4.28 mm to (127.2, 52.6)
- moved C33 4.08 mm to (108.2, 50.3)
- moved C31 3.82 mm to (145.8, 61.2), turned to 180 degrees
- moved C29 3.78 mm to (107.7, 69.5), turned to 180 degrees
- moved C28 1.84 mm to (88.7, 66.8), turned to 180 degrees
- moved C36 0.92 mm to (52.2, 54.8), turned to -90 degrees
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Routing:
- net /AN_SIG: track 0.00 -> 172.4 mm, vias 0 -> 6
- net /MTP_BIN_1: track 0.00 -> 153.4 mm, vias 0 -> 10
- net /MTP_BIN_0: track 0.00 -> 150.0 mm, vias 0 -> 9
- net /MTP_BIN_3: track 0.00 -> 99.3 mm, vias 0 -> 6
- net /MTP_BIN_2: track 0.00 -> 98.9 mm, vias 0 -> 6
- net /hesig32: track 0.00 -> 87.4 mm, vias 0 -> 1
- net /hesig30: track 0.00 -> 82.6 mm, vias 0 -> 1
- net /hesig29: track 0.00 -> 76.8 mm, vias 0 -> 1
- net /hesig31: track 0.00 -> 67.9 mm, vias 0 -> 1
- net /hesig35: track 0.00 -> 61.9 mm, vias 0 -> 1
- net /hesig28: track 0.00 -> 59.2 mm, vias 0 -> 1
- net NEOPIXEL_POWER: track 859.6 -> 914.5 mm, vias 27 -> 39
- net /hesig34: track 0.00 -> 40.4 mm, vias 0 -> 1
- net Net-(D27-DOUT): track 0.00 -> 35.0 mm, vias 0 -> 2
- net Net-(D26-DOUT): track 0.00 -> 28.3 mm
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