File: he_kbd/he_kbd.kicad_sch (KiCad schematic)
At the start: 53 parts, among them J1 AudioJack4

Commit message: I think it may be done... lets see how broken it is
Parts:
- added J2: Conn_01x08_Pin, Connector_PinHeader_1.27mm:PinHeader_1x08_P1.27mm_Horizontal, symbol Connector:Conn_01x08_Pin
Connections:
- net at AM2.2 (I7): now also J2.4 (Pin_4)
- net at AM2.21 (I10): now also J2.1 (Pin_1)
- net at AM2.22 (I9): now also J2.2 (Pin_2)
- net at AM2.23 (I8): now also J2.3 (Pin_3)
- net at AM2.3 (I6): now also J2.5 (Pin_5)
- net at AM2.4 (I5): now also J2.6 (Pin_6)
- net at AM2.5 (I4): now also J2.7 (Pin_7)
- net at AM2.6 (I3): now also J2.8 (Pin_8)
Changed lines of the file:
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@@
 	(wire
 		(pts
+			(xy 55.88 133.35) (xy 55.88 186.69)
+		)
+		(stroke
+			(width 0)
+			(type default)
+		)
+	)
+	(wire
+		(pts
 			(xy 246.38 59.69) (xy 246.38 73.66)
 		)
@@
 	(wire
 		(pts
+			(xy 59.69 181.61) (xy 73.66 181.61)
+		)
+		(stroke
+			(width 0)
+			(type default)
+		)
+	)
+	(wire
+		(pts
 			(xy 154.94 53.34) (xy 154.94 105.41)
 		)
@@
 	(wire
 		(pts
+			(xy 66.04 168.91) (xy 73.66 168.91)
+		)
+		(stroke
+			(width 0)
+			(type default)
+		)
+	)
+	(wire
+		(pts
 			(xy 236.22 49.53) (xy 236.22 101.6)
 		)
@@
 	(wire
 		(pts
+			(xy 60.96 179.07) (xy 73.66 179.07)
+		)
+		(stroke
+			(width 0)
+			(type default)
+		)
+	)
+	(wire
+		(pts
 			(xy 228.6 129.54) (xy 240.03 129.54)
 		)
@@
 	(wire
 		(pts
-			(xy 60.96 135.89) (xy 60.96 195.58)
+			(xy 60.96 135.89) (xy 60.96 179.07)
 		)
 		(stroke
@@
 	(wire
 		(pts
-			(xy 63.5 138.43) (xy 63.5 182.88)
+			(xy 63.5 138.43) (xy 63.5 173.99)
 		)
 		(stroke
@@
 	(wire
 		(pts
+			(xy 58.42 133.35) (xy 58.42 184.15)
+		)
+		(stroke
+			(width 0)
+			(type default)
+		)
+	)
+	(wire
+		(pts
 			(xy 228.6 58.42) (xy 220.98 58.42)
 		)
@@
 	(wire
 		(pts
+			(xy 59.69 134.62) (xy 59.69 181.61)
+		)
+		(stroke
+			(width 0)
+			(type default)
+		)
+	)
+	(wire
+		(pts
 			(xy 233.68 53.34) (xy 233.68 88.9)
 		)
@@
 	(wire
 		(pts
+			(xy 62.23 176.53) (xy 73.66 176.53)
+		)
+		(stroke
+			(width 0)
+			(type default)
+		)
+	)
+	(wire
+		(pts
 			(xy 238.76 50.8) (xy 237.49 50.8)
 		)
@@
 	(wire
 		(pts
+			(xy 64.77 171.45) (xy 73.66 171.45)
+		)
+		(stroke
+			(width 0)
+			(type default)
+		)
+	)
+	(wire
+		(pts
 			(xy 144.78 69.85) (xy 143.51 69.85)
 		)
@@
 	(wire
 		(pts
-			(xy 66.04 140.97) (xy 66.04 170.18)
+			(xy 66.04 140.97) (xy 66.04 168.91)
 		)
 		(stroke
@@
 	(wire
 		(pts
-			(xy 64.77 139.7) (xy 64.77 176.53)
+			(xy 64.77 139.7) (xy 64.77 171.45)
 		)
 		(stroke
@@
 	(wire
 		(pts
+			(xy 60.96 134.62) (xy 59.69 134.62)
+		)
+		(stroke
+			(width 0)
+			(type default)
+		)
+	)
+	(wire
+		(pts
 			(xy 173.99 60.96) (xy 162.56 60.96)
 		)
@@
 	(wire
 		(pts
+			(xy 63.5 173.99) (xy 73.66 173.99)
+		)
+		(stroke
+			(width 0)
+			(type default)
+		)
+	)
+	(wire
+		(pts
 			(xy 245.11 58.42) (xy 245.11 80.01)
 		)
@@
 	(wire
 		(pts
+			(xy 58.42 184.15) (xy 73.66 184.15)
+		)
+		(stroke
+			(width 0)
+			(type default)
+		)
+	)
+	(wire
+		(pts
 			(xy 105.41 52.07) (xy 105.41 54.61)
 		)
@@
 	(wire
 		(pts
+			(xy 55.88 186.69) (xy 73.66 186.69)
+		)
+		(stroke
+			(width 0)
+			(type default)
+		)
+	)
+	(wire
+		(pts
 			(xy 63.5 133.35) (xy 63.5 135.89)
 		)
@@
 	(wire
 		(pts
-			(xy 62.23 137.16) (xy 62.23 189.23)
+			(xy 62.23 137.16) (xy 62.23 176.53)
 		)
 		(stroke
@@
 	(wire
 		(pts
+			(xy 60.96 133.35) (xy 60.96 134.62)
+		)
+		(stroke
+			(width 0)
+			(type default)
+		)
+	)
+	(wire
+		(pts
 			(xy 231.14 49.53) (xy 231.14 53.34)
 		)
@@
 					(unit 1)
 				)
+			)
+		)
+	)
+	(symbol
+		(lib_id "Connector:Conn_01x08_Pin")
+		(at 78.74 179.07 180)
+		(unit 1)
+		(exclude_from_sim no)
+		(in_bom yes)
+		(on_board yes)
+		(dnp no)
+		(fields_autoplaced yes)
+		(property "Reference" "J2"
+			(at 80.01 176.5299 0)
+			(effects
+				(font
+					(size 1.27 1.27)
+				)
+				(justify right)
+			)
+		)
+		(property "Value" "Conn_01x08_Pin"
+			(at 80.01 179.0699 0)
+			(effects
+				(font
+					(size 1.27 1.27)
+				)
+				(justify right)
+			)
+		)
+		(property "Footprint" "Connector_PinHeader_1.27mm:PinHeader_1x08_P1.27mm_Horizontal"
+			(at 78.74 179.07 0)
+			(effects
+				(font
+					(size 1.27 1.27)
+				)
+				(hide yes)
+			)
+		)
+		(property "Datasheet" "~"
+			(at 78.74 179.07 0)
+			(effects
+				(font
+					(size 1.27 1.27)
+				)
+				(hide yes)
+			)
+		)
+		(property "Description" "Generic connector, single row, 01x08, script generated"
+			(at 78.74 179.07 0)
+			(effects
+				(font
+					(size 1.27 1.27)
+				)
+				(hide yes)
+			)
+		)
+		(pin "6"
+		)
+		(pin "2"
+		)
+		(pin "5"
+		)
+		(pin "4"
+		)
+		(pin "7"
+		)
+		(pin "8"
+		)
+		(pin "3"
+		)
+		(pin "1"
+		)
+		(instances
+			(project ""
+				(path "/ec6e5a97-af17-41bd-90dd-eb7235b0e08a"
+					(reference "J2")
+					(unit 1)
+				)

Commit message: tidying up schematic
Connections:
- net ANALOGUE_VIN: now also A1.36 (3V3); no longer A1.35 (ADC_VREF)
- net GND: now also C43.2, C44.2, C45.2, C46.2, C47.2, C48.2, C49.2, C50.2, HE_1.3 (GND), HE_10.3 (GND), HE_11.3 (GND), HE_12.3 (GND), HE_13.3 (GND), HE_14.3 (GND), HE_15.3 (GND), HE_16.3 (GND), HE_17.3 (GND), HE_18.3 (GND), HE_19.3 (GND), HE_2.3 (GND), HE_20.3 (GND), HE_21.3 (GND), HE_22.3 (GND), HE_23.3 (GND), HE_24.3 (GND), HE_25.3 (GND), HE_26.3 (GND), HE_27.3 (GND), HE_28.3 (GND), HE_29.3 (GND), HE_3.3 (GND), HE_30.3 (GND), HE_31.3 (GND), HE_32.3 (GND), HE_33.3 (GND), HE_34.3 (GND), HE_35.3 (GND), HE_4.3 (GND), HE_5.3 (GND), HE_6.3 (GND), HE_7.3 (GND), HE_8.3 (GND), HE_9.3 (GND)
- removed net ANALOGUE_GND: A1.33 (AGND), C43.2, C44.2, C45.2, C46.2, C47.2, C48.2, C49.2, C50.2, HE_1.3 (GND), HE_10.3 (GND), HE_11.3 (GND), HE_12.3 (GND), HE_13.3 (GND), HE_14.3 (GND), HE_15.3 (GND), HE_16.3 (GND), HE_17.3 (GND), HE_18.3 (GND), HE_19.3 (GND), HE_2.3 (GND), HE_20.3 (GND), HE_21.3 (GND), HE_22.3 (GND), HE_23.3 (GND), HE_24.3 (GND), HE_25.3 (GND), HE_26.3 (GND), HE_27.3 (GND), HE_28.3 (GND), HE_29.3 (GND), HE_3.3 (GND), HE_30.3 (GND), HE_31.3 (GND), HE_32.3 (GND), HE_33.3 (GND), HE_34.3 (GND), HE_35.3 (GND), HE_4.3 (GND), HE_5.3 (GND), HE_6.3 (GND), HE_7.3 (GND), HE_8.3 (GND), HE_9.3 (GND)
Other:
- note added: "Hall effect Sensors / Transistors"
- note added: "Multiplexers"
- moved on the sheet: A1, AM0, AM1, AM2, HE_1, HE_10, HE_11, HE_12, HE_13, HE_14, HE_15, HE_16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
